File: Titulador.sch (KiCad schematic (older format))
At the start: 43 parts, among them J1 1x2_F, J2 1x2_F, J3 1x6_F, J4 Conn_01x06_Female, J5 1x5_F, J6 1x4_F, J7 1x2_F, J8 Conn_02x03_Odd_Even, Q1 BC548, SW1 SW_DIP_x04, U1 LM7805_TO220, U2 ESP32-DEVKITC-32D, U3 ATmega328P-PU, Y1 Crystal

Commit message: Se finaliza primera version esquematico y PCB
Parts:
- removed J5: 1x5_F, Connector_PinSocket_2.54mm:PinSocket_1x05_P2.54mm_Vertical, symbol Connector:Conn_01x05_Female
- removed R12: 33K, Resistor_THT:R_Axial_DIN0207_L6.3mm_D2.5mm_P7.62mm_Horizontal, symbol Device:R
- removed R13: 18K, Resistor_THT:R_Axial_DIN0207_L6.3mm_D2.5mm_P7.62mm_Horizontal, symbol Device:R
- added J5: 1x4_F, Connector_PinSocket_2.54mm:PinSocket_1x04_P2.54mm_Vertical, symbol Connector:Conn_01x04_Female
- C2, C3, C4, C5: footprint (none) -> Capacitor_THT:C_Axial_L5.1mm_D3.1mm_P7.50mm_Horizontal
- C6, C7: value C -> 22nF; footprint (none) -> Capacitor_THT:C_Axial_L5.1mm_D3.1mm_P7.50mm_Horizontal
- D2: value D -> 1N4148; footprint (none) -> Diode_THT:D_A-405_P7.62mm_Horizontal
- J4: value Conn_01x06_Female -> 1x6_F; footprint (none) -> Connector_PinHeader_2.54mm:PinHeader_1x06_P2.54mm_Vertical
- J8: value Conn_02x03_Odd_Even -> 2x3_Odd_Even; footprint (none) -> Connector_PinHeader_2.54mm:PinHeader_2x03_P2.54mm_Vertical
- U1: footprint Package_TO_SOT_THT:TO-220-3_Vertical -> Package_TO_SOT_THT:TO-220F-3_Horizontal_TabDown
- Y1: value Crystal -> 16MHz; footprint (none) -> Crystal:Crystal_HC18-U_Vertical
- renumbered R14 to R12
Connections:
- net DirPAP: now also U2.11 (IO27); no longer U2.22 (IO22)
- net HMISO: now also U2.34 (IO2)
- net StepPAP: now also U2.13 (IO12); no longer U2.25 (IO21)
- net at U2.10 (IO26): now also J5.4 (Pin_4); no longer J4.4 (Pin_4)
- net at J4.5 (Pin_5): now also U2.25 (IO21); no longer U2.11 (IO27)
- net at J4.6 (Pin_6): now also U2.22 (IO22); no longer U2.13 (IO12)
- net at U2.27 (IO19): now also J4.4 (Pin_4)
- net at U2.28 (IO18): now also J4.3 (Pin_3)
- net at U2.31 (IO16): now also J4.2 (Pin_2)
- net at U2.33 (IO0): now also J4.1 (Pin_1)
- net at U2.7 (IO32): now also J5.1 (Pin_1); no longer J4.1 (Pin_1)
- net at U2.8 (IO33): now also J5.2 (Pin_2); no longer J4.2 (Pin_2)
- net at U2.9 (IO25): now also J5.3 (Pin_3); no longer J4.3 (Pin_3)
- net at A1.3 (A2): now also J6.1 (Pin_1); no longer J6.3 (Pin_3)
- net at A1.4 (A1): now also J6.2 (Pin_2); no longer J6.4 (Pin_4)
- net at A1.5 (B1): now also J6.3 (Pin_3); no longer J6.2 (Pin_2)
- net at A1.6 (B2): now also J6.4 (Pin_4); no longer J6.1 (Pin_1)
- net +3V3: no longer names the net of U2.1 (3V3)
- net +3V3: no longer A2.27 (3.3V)
- no-connect marks 17 -> 20
Other:
- note added: "ICSP"
- moved on the sheet: J4
